Commit message: full urdf completed

File: src/soapPackage/description/robot_core.xacro (robot description, xacro)
@@ -31,3 +31,33 @@
         </visual>
     </link>
+    <!-- LEFT PROPELLER -->
+    <joint name="left_propeller_joint" type="continuous">
+        <parent link="chassis"/>
+        <child link="left_propeller"/>
+        <origin xyz="-.03 -0.1 0.02" rpy="0 ${pi/2} 0"/>
+        <axis xyz="0 0 1"/>
+    </joint>
+    <link name="left_propeller">
+        <visual>
+            <geometry>
+                <cylinder radius=".02" length=".06"/>
+            </geometry>
+            <material name="orange"/>
+        </visual>
+    </link>
+    <!-- RIGHT PROPELLER-->
+    <joint name="right_propeller_joint" type="continuous">
+        <parent link="chassis"/>
+        <child link="right_propeller"/>
+        <origin xyz="-.03 0.1 0.02" rpy="0 ${pi/2} 0"/>
+        <axis xyz="0 0 1"/>
+    </joint>
+    <link name="right_propeller">
+        <visual>
+            <geometry>
+                <cylinder radius=".02" length=".06"/>
+            </geometry>
+            <material name="orange"/>
+        </visual>
+    </link>
 </robot>

Commit message: interia stuff added

File: src/soapPackage/description/robot_core.xacro (robot description, xacro)
@@ -30,4 +30,13 @@
             <material name="white"/>
         </visual>
+        <collision>
+            <origin xyz="0.15 0 0.075"/>
+            <geometry>
+                <box size="0.3 0.3 0.15"/>
+            </geometry>
+        </collision>
+        <xacro:inertial_box mass="0.7" x="0.3" y="0.3" z="0.15">
+            <origin xyz="0.15 0 0.075"/>
+        </xacro:inertial_box>
     </link>
     <!-- LEFT PROPELLER -->
@@ -45,5 +54,13 @@
             <material name="orange"/>
         </visual>
+        <collision>
+            <geometry>
+                <cylinder radius=".02" length=".06"/>
+            </geometry>
+        </collision>
     </link>
+    <xacro:inertial_cylinder mass=".03" x="-0.3" y="-0.1" z="0.02">
+        <origin xyz="0 0 0" rpy="0 0 0"/>
+    </xacro:inertial_cylinder>
     <!-- RIGHT PROPELLER-->
     <joint name="right_propeller_joint" type="continuous">
@@ -60,4 +77,12 @@
             <material name="orange"/>
         </visual>
+        <collision>
+            <geometry>
+                <cylinder radius=".02" length=".06"/>
+            </geometry>
+        </collision>
+        <xacro:inertial_cylinder mass=".03" x="0.3" y="0.1" z="0.02">
+        <origin xyz="0 0 0" rpy="0 0 0"/>
+    </xacro:inertial_cylinder>
     </link>
 </robot>

Commit message: need to smooth out drive

File: src/soapPackage/description/robot_core.xacro (robot description, xacro)
@@ -1,4 +1,5 @@
 <?xml version="1.0"?>
 <robot xmlns:xacro="http://www.ros.org/wiki/xacro" >
+    <xacro:include filename="inertial_macros.xacro"/>
     <material name="white">
         <color rgba="1 1 1 1" />
@@ -40,4 +41,7 @@
         </xacro:inertial_box>
     </link>
+    <gazebo reference="chassis">
+        <material>Gazebo/White</material>
+    </gazebo>
     <!-- LEFT PROPELLER -->
     <joint name="left_propeller_joint" type="continuous">
@@ -59,8 +63,11 @@
             </geometry>
         </collision>
+        <xacro:inertial_cylinder mass=".03" length=".06" radius=".02">
+            <origin xyz="0 0 0" rpy="0 0 0"/>
+        </xacro:inertial_cylinder>
     </link>
-    <xacro:inertial_cylinder mass=".03" x="-0.3" y="-0.1" z="0.02">
-        <origin xyz="0 0 0" rpy="0 0 0"/>
-    </xacro:inertial_cylinder>
+    <gazebo reference="left_propeller">
+        <material>Gazebo/Orange</material>
+    </gazebo>
     <!-- RIGHT PROPELLER-->
     <joint name="right_propeller_joint" type="continuous">
@@ -82,7 +89,102 @@
             </geometry>
         </collision>
-        <xacro:inertial_cylinder mass=".03" x="0.3" y="0.1" z="0.02">
-        <origin xyz="0 0 0" rpy="0 0 0"/>
-    </xacro:inertial_cylinder>
+        <xacro:inertial_cylinder mass=".03" length=".06" radius=".02">
+            <origin xyz="0 0 0" rpy="0 0 0"/>
+        </xacro:inertial_cylinder>
     </link>
+    <gazebo reference="right_propeller">
+        <material>Gazebo/Orange</material>
+    </gazebo>
+    <!-- LEFT WHEEL LINK -->
+    <joint name="left_wheel_joint" type="continuous">
+        <parent link="base_link"/>
+        <child link="left_wheel"/>
+        <origin xyz="0 0.175 0" rpy="-${pi/2} 0 0" />
+        <axis xyz="0 0 1"/>
+    </joint>
+    <link name="left_wheel">
+        <visual>
+            <geometry>
+                <cylinder radius="0.05" length="0.04"/>
+            </geometry>
+            <material name="blue"/>
+        </visual>
+        <collision>
+            <geometry>
+                <cylinder radius="0.05" length="0.04"/>
+            </geometry>
+        </collision>
+        <xacro:inertial_cylinder mass="0.1" length="0.04" radius="0.05">
+            <origin xyz="0 0 0" rpy="0 0 0"/>
+        </xacro:inertial_cylinder>
+    </link>
+    <gazebo reference="left_wheel">
+        <material>
+            <script>
+              <name>Gazebo/BlueTransparent</name>
+              <uri>file://media/materials/scripts/gazebo.material</uri>
+            </script>
+          </material>
+    </gazebo>
+    <!-- RIGHT WHEEL LINK -->
+    <joint name="right_wheel_joint" type="continuous">
+        <parent link="base_link"/>
+        <child link="right_wheel"/>
+        <origin xyz="0 -0.175 0" rpy="${pi/2} 0 0" />
+        <axis xyz="0 0 -1"/>
+    </joint>
+    <link name="right_wheel">
+        <visual>
+            <geometry>
+                <cylinder radius="0.05" length="0.04"/>
+            </geometry>
+            <material name="blue"/>
+        </visual>
+        <collision>
+            <geometry>
+                <cylinder radius="0.05" length="0.04"/>
+            </geometry>
+        </collision>
+        <xacro:inertial_cylinder mass="0.1" length="0.04" radius="0.05">
+            <origin xyz="0 0 0" rpy="0 0 0"/>
+        </xacro:inertial_cylinder>
+    </link>
+    <gazebo reference="right_wheel">
+        <material>
+            <script>
+              <name>Gazebo/BlueTransparent</name>
+              <uri>file://media/materials/scripts/gazebo.material</uri>
+            </script>
+          </material>
+    </gazebo>
+    <!-- CASTER WHEEL LINK -->
+    <joint name="caster_wheel_joint" type="fixed">
+        <parent link="chassis"/>
+        <child link="caster_wheel"/>
+        <origin xyz="0.24 0 0"/>
+    </joint>
+    <link name="caster_wheel">
+        <visual>
+            <geometry>
+                <sphere radius="0.05"/>
+            </geometry>
+            <material name="black"/>
+        </visual>
+        <collision>
+            <geometry>
+                <sphere radius="0.05"/>
+            </geometry>
+        </collision>
+        <xacro:inertial_sphere mass="0.1" radius="0.05">
+            <origin xyz="0 0 0" rpy="0 0 0"/>
+        </xacro:inertial_sphere>
+    </link>
+    <gazebo reference="caster_wheel">
+        <material>
+            <script>
+              <name>Gazebo/BlueTransparent</name>
+              <uri>file://media/materials/scripts/gazebo.material</uri>
+            </script>
+          </material>
+    </gazebo>
 </robot>
